File: lmh7324/quad.sch (KiCad schematic (older format))
At the start: 47 parts, among them IC1 lmh7324

Commit message: Trying mass-edit of net names
Parts:
- removed C1, C2, C4: 10uF, symbol Device:C
- removed C24, C25: 10n, symbol Device:C
- removed C26, C27, C28, C29, C30, C31, C9: 100n, symbol Device:C
- IC1: symbol lmh732x:lmh7324 -> mso5k-la-rescue:lmh7324-lmh732x

Commit message: completed core layout of 16 channel lmh7324 design
Parts:
- removed IC1: lmh7324, symbol mso5k-la-rescue:lmh7324-lmh732x
- removed RN1: 200, symbol Device:R_Pack08
- removed RN2: 49R9, symbol Device:R_Pack08
- added IC201: lmh7324, Package_DFN_QFN:QFN-32-1EP_5x5mm_P0.5mm_EP3.1x3.1mm_ThermalVias, symbol lmh7324:lmh7324
- added RN201, RN203: 200, Resistors_SMD.pretty:R_Array_Convex_4x0603, symbol Device:R_Pack04
- added RN202, RN204: 49R9, Resistors_SMD.pretty:R_Array_Convex_4x0603, symbol Device:R_Pack04
- C401: renamed from C3; footprint (none) -> Capacitors_SMD.pretty:C_0603
- C402: renamed from C5; footprint (none) -> Capacitors_SMD.pretty:C_0603
- C403: renamed from C6; footprint (none) -> Capacitors_SMD.pretty:C_0603
- C404: renamed from C8; footprint (none) -> Capacitors_SMD.pretty:C_0603
- C405: renamed from C10; footprint (none) -> Capacitors_SMD.pretty:C_0603
- C406: renamed from C11; footprint (none) -> Capacitors_SMD.pretty:C_0603
- C407: renamed from C12; footprint (none) -> Capacitors_SMD.pretty:C_0603
- C408: renamed from C13; footprint (none) -> Capacitors_SMD.pretty:C_0603
- C409: renamed from C14; footprint (none) -> Capacitors_SMD.pretty:C_0603
- C410: renamed from C16; footprint (none) -> Capacitors_SMD.pretty:C_0603
- C411: renamed from C15; footprint (none) -> Capacitors_SMD.pretty:C_0603
- C412: renamed from C17; footprint (none) -> Capacitors_SMD.pretty:C_0603
- C413: renamed from C18; footprint (none) -> Capacitors_SMD.pretty:C_0603
- C414: renamed from C19; footprint (none) -> Capacitors_SMD.pretty:C_0603
- C415: renamed from C20; footprint (none) -> Capacitors_SMD.pretty:C_0603
- C416: renamed from C22; footprint (none) -> Capacitors_SMD.pretty:C_0603
- R401: renamed from R1; footprint (none) -> Resistors_SMD.pretty:R_0603
- R402: renamed from R2; footprint (none) -> Resistors_SMD.pretty:R_0603
- R403: renamed from R3; footprint (none) -> Resistors_SMD.pretty:R_0603
- R404: renamed from R4; footprint (none) -> Resistors_SMD.pretty:R_0603
- R405: renamed from R5; footprint (none) -> Resistors_SMD.pretty:R_0603
- R406: renamed from R6; footprint (none) -> Resistors_SMD.pretty:R_0603
- R407: renamed from R7; footprint (none) -> Resistors_SMD.pretty:R_0603
- R408: renamed from R8; footprint (none) -> Resistors_SMD.pretty:R_0603
- R409: renamed from R17; footprint (none) -> Resistors_SMD.pretty:R_0603
- R410: renamed from R18; footprint (none) -> Resistors_SMD.pretty:R_0603
- R411: renamed from R19; footprint (none) -> Resistors_SMD.pretty:R_0603
- R412: renamed from R20; footprint (none) -> Resistors_SMD.pretty:R_0603
- R413: renamed from R21; footprint (none) -> Resistors_SMD.pretty:R_0603
- R414: renamed from R22; footprint (none) -> Resistors_SMD.pretty:R_0603
- R415: renamed from R23; footprint (none) -> Resistors_SMD.pretty:R_0603
- R416: renamed from R24; footprint (none) -> Resistors_SMD.pretty:R_0603
Connections:
- net +2V5: now also IC201.1 (VCCO), IC201.17 (VCCO), IC201.24 (VCCO), IC201.8 (VCCO)
- net +4V: now also IC201.16 (VCCI), IC201.25 (VCCI), IC201.32 (VCCI), IC201.9 (VCCI)
- net -2V5: now also IC201.12 (VEE), IC201.13 (VEE), IC201.20 (VEE), IC201.21 (VEE), IC201.28 (VEE), IC201.29 (VEE), IC201.4 (VEE), IC201.5 (VEE)
- net GND: now also IC201.33 (pad), IC201.33 (pad), IC201.33 (pad), IC201.33 (pad), RN201.1 (R1.1), RN201.2 (R2.1), RN201.3 (R3.1), RN201.4 (R4.1), RN203.1 (R1.1), RN203.2 (R2.1), RN203.3 (R3.1), RN203.4 (R4.1)
- net Vref: now also IC201.10 (In-), IC201.15 (In-), IC201.26 (In-), IC201.31 (In-)
- net at C401.1, C403.1, R405.1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: now also IC201.27 (in+)
- net at C402.1, C404.1, R406.1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: now also IC201.14 (in+)
- net at C413.1, C415.1, R413.1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: now also IC201.11 (in+)
- net at C414.1, C416.1, R414.1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: now also IC201.30 (in+)
- new net A+: IC201.22 (Q), RN201.7 (R2.2), RN202.2 (R2.1)
- new net A-: IC201.23 (~Q), RN201.8 (R1.2), RN202.1 (R1.1)
- new net B+: IC201.19 (Q), RN201.6 (R3.2), RN202.3 (R3.1)
- new net B-: IC201.18 (~Q), RN201.5 (R4.2), RN202.4 (R4.1)
- new net C+: IC201.6 (Q), RN203.7 (R2.2), RN204.2 (R2.1)
- new net C-: IC201.7 (~Q), RN203.8 (R1.2), RN204.1 (R1.1)
- new net D+: IC201.3 (Q), RN203.6 (R3.2), RN204.3 (R3.1)
- new net D-: IC201.2 (~Q), RN203.5 (R4.2), RN204.4 (R4.1)
- new net OutA+: RN202.7 (R2.2)
- new net OutA-: RN202.8 (R1.2)
- new net OutB+: RN202.6 (R3.2)
- new net OutB-: RN202.5 (R4.2)
- new net OutC+: RN204.7 (R2.2)
- new net OutC-: RN204.8 (R1.2)
- new net OutD+: RN204.6 (R3.2)
- new net OutD-: RN204.5 (R4.2)
