File: lmh7324-8ch/leds.sch (KiCad schematic (older format))
At the start: 17 parts, among them U401 ATtiny85-20SU

Commit message: Added fixes for E1 and E2
Parts:
- removed R417: 10k, Resistor_SMD:R_0603_1608Metric, symbol Device:R
Connections:
- net PB0: now reaches D401.1 (K), D402.2 (A), R418.1
- net PB0: now also D407.2 (A), D408.1 (K)
- net PB1: now reaches D401.2 (A), D402.1 (K), D403.1 (K), D404.2 (A), D409.2 (A), D410.1 (K), R419.1
- net PB2: now reaches D403.2 (A), D404.1 (K), D405.1 (K), D406.2 (A), R420.1
- net PB2: no longer D407.2 (A), D408.1 (K)
- net PB3: now reaches D405.2 (A), D406.1 (K), D407.1 (K), D408.2 (A), D409.1 (K), D410.2 (A), R421.1
Other:
- note added: "Note: Programming via SOIC clip, which connects to:\nRESET (pin 1) \nSCK (pin 7) aka PB2\nMOSI (pin 5) aka PB0\nMISO (pin 6) aka PB1\nVCC (pin 8)\nGND (pin 4)"
Changed lines of the file:
@@
 Wire Wire Line
 	5400 3200 5250 3200
-$Comp
-L Device:R R417
-U 1 1 5C610201
-P 5000 3750
-F 0 "R417" V 5100 3650 50  0000 C CNN
-F 1 "10k" V 5000 3750 50  0000 C CNN
-F 2 "Resistor_SMD:R_0603_1608Metric" V 4930 3750 50  0001 C CNN
-F 3 "~" H 5000 3750 50  0001 C CNN
-	1    5000 3750
-	0    1    1    0
-$EndComp
-Wire Wire Line
-	4850 3750 4650 3750
 Wire Wire Line
 	4650 3700 4650 3750
@@
 Wire Wire Line
 	4650 3750 4650 3850
-Wire Wire Line
-	5150 3750 5300 3750
-Wire Wire Line
-	5300 3750 5300 3300
-Wire Wire Line
-	5300 3300 5250 3300
 $Comp
 L Device:LED D401
@@
 	6650 2300 6700 2300
 Wire Wire Line
-	6700 2300 6700 2400
-Wire Wire Line
 	6700 2500 6650 2500
 Wire Wire Line
@@
 	6650 3100 6700 3100
 Wire Wire Line
-	6700 3100 6700 3200
-Wire Wire Line
 	6700 3300 6650 3300
 Wire Wire Line
@@
 Connection ~ 6700 2100
 Connection ~ 6300 2300
-Wire Wire Line
-	6700 2500 6700 2600
-Wire Wire Line
-	6700 2600 6300 2600
-Wire Wire Line
-	6300 2600 6300 2700
-Connection ~ 6700 2500
 Connection ~ 6300 2700
 Wire Wire Line
@@
 Connection ~ 6700 2900
 Connection ~ 6300 3100
-Wire Wire Line
-	6700 3200 6950 3200
-Wire Wire Line
-	6950 3200 6950 2400
-Wire Wire Line
-	6950 2400 6700 2400
-Connection ~ 6700 3200
-Wire Wire Line
-	6700 3200 6700 3300
-Connection ~ 6700 2400
-Wire Wire Line
-	6700 2400 6700 2500
 Wire Wire Line
 	6700 3600 7000 3600
@@
 Wire Wire Line
 	3850 3750 4650 3750
+Wire Wire Line
+	6700 2300 6700 2500
+Wire Wire Line
+	6700 3100 6700 3200
+Wire Wire Line
+	6700 3200 6950 3200
+Connection ~ 6700 3200
+Wire Wire Line
+	6700 3200 6700 3300
+Wire Wire Line
+	6300 2600 6300 2700
+Connection ~ 6700 2500
+Wire Wire Line
+	6700 2500 6700 2600
+Wire Wire Line
+	6700 2600 6300 2600
+Wire Wire Line
+	6950 3200 6950 1800
+Wire Wire Line
+	6300 1800 6300 1900
+Wire Wire Line
+	6950 1800 6300 1800
+Text Label 6000 1900 0    50   ~ 0
+PB0
+Text Label 6100 2300 0    50   ~ 0
+PB1
+Text Label 6150 2700 0    50   ~ 0
+PB2
+Text Label 6100 3100 0    50   ~ 0
+PB3
+Text Notes 3800 4750 0    50   ~ 0
+Note: Programming via SOIC clip, which connects to:\nRESET (pin 1) \nSCK (pin 7) aka PB2\nMOSI (pin 5) aka PB0\nMISO (pin 6) aka PB1\nVCC (pin 8)\nGND (pin 4)
 $EndSCHEMATC

Commit message: Cleaning up
Connections:
- net ~Reset: now reaches U401.1 (~RESET~/PB5)
Changed lines of the file:
@@
 Text Notes 3800 4750 0    50   ~ 0
 Note: Programming via SOIC clip, which connects to:\nRESET (pin 1) \nSCK (pin 7) aka PB2\nMOSI (pin 5) aka PB0\nMISO (pin 6) aka PB1\nVCC (pin 8)\nGND (pin 4)
+Text GLabel 5400 3300 2    50   Input ~ 0
+~Reset
+Wire Wire Line
+	5400 3300 5250 3300
 $EndSCHEMATC
