File: lmh7324-8ch/mso5k-la.kicad_pcb (KiCad board)
At the start: 4 copper layers, 40 x 42 mm, 126 parts, among them IC201 lmh7324, IC401 lmh7324, J101 out, J102 in, J103 3mm, J104 3mm, J105 3mm, J106 3mm, U401 ATtiny85-20SU

Commit message: Cleaning up
Parts:
- removed G***: LOGO, lmh7324-8ch:qrcode
- removed R417: 10k, Resistor_SMD:R_0603_1608Metric
- moved J106 50.6 mm to (19.3, 18.2), turned to 180 degrees
- moved J103 50.1 mm to (19.3, 54.2), turned to 180 degrees
- moved J104 48.9 mm to (53.3, 18.2), turned to 180 degrees
- moved J105 48.4 mm to (53.3, 54.2), turned to 180 degrees
- moved C102 43.9 mm to (24.9, 18.0), turned to 180 degrees
- moved D401 42.3 mm to (50.9, 22.5), turned to 90 degrees
- moved J102 41.0 mm to (45.1, 55.1), turned to 270 degrees
- moved D410 40.6 mm to (50.9, 49.9), turned to 90 degrees
- moved R421 40.2 mm to (22.0, 47.1), turned to 180 degrees
- moved C104 40.2 mm to (22.2, 23.6), turned to 90 degrees
- moved C417 39.5 mm to (22.2, 26.7), turned to 270 degrees
- moved D402 38.6 mm to (50.9, 25.5), turned to 90 degrees
- moved R418 38.2 mm to (22.0, 45.5), turned to 180 degrees
- moved D409 37.1 mm to (50.9, 46.9), turned to 90 degrees
- moved R419 36.4 mm to (22.0, 43.9), turned to 180 degrees
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Connections:
- net Net-(D401-Pad1) renamed /LEDs/PB0
- net Net-(D401-Pad2) renamed /LEDs/PB1
- net Net-(D403-Pad2) renamed /LEDs/PB2
- net Net-(D405-Pad2) renamed /LEDs/PB3
- U401 pad 1: Net-(R417-Pad1) -> ~Reset
Routing:
- net +4V: track 86.4 -> 127.4 mm, vias 19 -> 21
- net ~Reset: track 0.00 -> 26.2 mm, vias 0 -> 1
- net -2V5: track 118.2 -> 135.9 mm, vias 16 -> 18
- net /LEDs/PB0: track 65.5 -> 52.0 mm, vias 4 -> 2
- net Net-(R420-Pad2): track 6.98 -> 19.4 mm, vias 0 -> 1
- net +2V5: track 155.6 -> 166.9 mm, vias 22 -> 23
- net Net-(R417-Pad1): track 11.0 -> 0.00 mm, vias 2 -> 0
- net Net-(R419-Pad2): track 8.96 -> 19.5 mm, vias 0 -> 1
- net /LEDs/PB2: track 53.2 -> 43.0 mm, vias 2 -> 4
- net /LEDs/PB3: track 54.4 -> 45.4 mm, vias 6 -> 3
- net Net-(R418-Pad2): track 11.1 -> 20.0 mm
- net /LEDs/PB1: track 68.2 -> 61.5 mm, vias 6 -> 3
- net Vref: track 128.5 -> 122.9 mm
- net Net-(R421-Pad2): track 21.7 -> 17.6 mm
- net /Ch 4-7/C+: track 14.6 -> 13.9 mm
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- removed copper zone on 3_Misc, net +4V
Other:
- board text added: "+"
- board text added: "-"
- board text added: "-1.3V ECL"
- board text added: "0.9V CMOS @1.8V"
- board text added: "1.2V LVDS"
- board text added: "1.4V TTL"
- board text added: "1.65V CMOS @3.3V"
- board text added: "2.5V CMOS @5V"
- board text added: "3.7V PECL"
- board text added: "MISO"
- board text added: "MOSI"
- board text added: "SCK"
- board text added: "~RESET"
- board text removed: "-1.3V"
- board text removed: "0.9V"
- board text removed: "1.2V"
- board text removed: "1.4V"
- board text removed: "1.65V"
- board text removed: "2.5V"
- board text removed: "3.7V"
- board text removed: "CMOS @1.8V"
- board text removed: "CMOS @3.3V"
- board text removed: "CMOS @5V"
- board text removed: "ECL"
- board text removed: "LVDS"
- board text removed: "PECL"
- board text removed: "TTL"
